File: aart-brake-kicad/aart_brake.kicad_sch (KiCad schematic)
At the start: 0 parts

Commit message: Debug pins
Other:
- note added: "=== BOOT0 BUTTON (J12) ==="
- note added: "=== NRST BUTTON (J13) ==="
- note added: "=== SWD DEBUG / FLASH HEADER (J10) ==="
- note added: "=== UART DEBUG / BOOTLOADER (J11) ==="
- note added: "COMPONENT LIST (Rev 9): U1 STM32G041K6U6 QFN-32 U2 AMS1117-3.3 SOT-223 GD1 UCC27524 SOT-23-5 (brake gate driver) GD2 UCC27524 SOT-23-5 (keep-alive gate driver) Q1 IRLB3034 D2PAK (N-ch brake FET) Q2 IRF9Z34N D2PAK (P-ch keep-alive FET) D1 P6KE18CA SMB (TVS BIDIRECTIONAL - CA suffix essential) D2 SS310 SMB (Q1 catch - 100V required) D3 SS310 SMB (Q2 catch - 100V required) D4 MBRS360/SS54 SMB (mode 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"
- note added: "J12: momentary button PB8/BOOT0 to 3.3V Hold J12 + press J13 NRST = ROM bootloader entry Flash via J11 UART: stm32flash -w aart_brake.bin /dev/ttyUSB0"
- note added: "J13: momentary button NRST to GND Press while holding J12 BOOT0 to enter bootloader. Release J13 first, then release J12."
- note added: "PLACEMENT GUIDE: Top-left: Power (J1 rail, F1, D1, U2, C1-C4) Top-centre: SWD J10 | UART J11 Left-mid: Inputs (pot, toggle, capture btn, dividers) Below-left: BOOT0 J12 | NRST J13 Centre: MCU U1, C5-C7, R1 Right-upper: Brake FET (GD1, R2, R3, Q1, D2) Right-lower: Keep-alive FET (GD2, R4, Q2, D3, D4) Far-right: Track banana J1-J6 Below MCU: Status LED R12 D5 R2 pull-up: on GD1 INA input - NOT on Q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"
- note added: "POT MAPPING (all modes): CCW => min brake (~8 ohm) CW => max brake (dead short) Mode A: centre = dead short CW past centre = positive anti-brake 0-2V"
- note added: "Pin 1: SWDIO (PA13) Pin 2: SWDCLK (PA14) Pin 3: GND Pin 4: +3.3V (optional) 2.54mm 4-pin header. Match your ST-Link V2/V3 pinout."
- note added: "Pin 1: TX PA9 (-> RX of USB-UART adapter) Pin 2: RX PA10 (-> TX of USB-UART adapter) Pin 3: GND 115200 8N1, 3.3V logic. Telemetry CSV at 100ms interval. Also used by ROM bootloader (hold BOOT0 + press NRST)."
- note added: "Q2: P-ch high-side keep-alive FET TIM3_CH2 normal polarity CCR=0 => FET OFF CCR=400 => ~2V injected at 16V rail"
- note removed: "=== POWER SUPPLY ==="
- note removed: "COMPONENT LIST: U1 STM32G041K6U6 QFN-32 U2 AMS1117-3.3 SOT-223 GD1 UCC27524 SOT-23-5 (brake gate driver) GD2 UCC27524 SOT-23-5 (keep-alive gate driver) Q1 IRLB3034 D2PAK (N-ch brake FET) Q2 IRF9Z34N D2PAK (P-ch keep-alive FET) D1 P6KE15A SMB (TVS rail clamp) D2 SS34 SMB (Q1 catch diode) D3 SS34 SMB (Q2 catch diode) D4 SS34 SMB (mode C series protection) D5 LED Red 0805 (status LED) F1 Polyfuse 25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"
- note removed: "POT MAPPING (all modes): CCW => min brake (~8 ohm) CW => max brake (dead short) Mode A: centre = dead short CW past centre = antibrake 0-3V"
- note removed: "Q2: P-ch high-side keep-alive FET TIM3_CH2 normal polarity CCR=0 => FET OFF CCR=774 => ~3V injected"
Changed lines of the file:
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@@
   (global_label "GND" (shape passive) (at 222.25 120.65 90)
     (effects (font (size 1.27 1.27)) (justify right)))
-  (text "=== POWER SUPPLY ===" (at 15.24 15.24 0)
-    (effects (font (size 1.5 1.5) bold)))
+  (global_label "SWDIO" (shape input) (at 120.65 55.88 0)
+    (effects (font (size 1.27 1.27)) (justify left)))
+  (global_label "SWDCLK" (shape input) (at 120.65 58.42 0)
+    (effects (font (size 1.27 1.27)) (justify left)))
+  (global_label "SWDIO" (shape output) (at 86.36 68.58 180)
+    (effects (font (size 1.27 1.27)) (justify right)))
+  (global_label "SWDCLK" (shape output) (at 86.36 71.12 180)
+    (effects (font (size 1.27 1.27)) (justify right)))
+  (wire (pts (xy 120.65 55.88) (xy 132.08 55.88)))
+  (wire (pts (xy 120.65 58.42) (xy 132.08 58.42)))
+  (wire (pts (xy 132.08 55.88) (xy 132.08 63.5)))
+  (wire (pts (xy 132.08 58.42) (xy 132.08 63.5)))
+  (wire (pts (xy 132.08 63.5) (xy 139.7 63.5)))
+  (wire (pts (xy 139.7 55.88) (xy 139.7 66.04)))
+  (wire (pts (xy 139.7 66.04) (xy 144.78 66.04)))
+  (global_label "GND" (shape passive) (at 144.78 63.5 0)
+    (effects (font (size 1.27 1.27)) (justify left)))
+  (global_label "+3V3" (shape passive) (at 139.7 53.34 270)
+    (effects (font (size 1.27 1.27)) (justify left)))
+  (global_label "UART_TX" (shape output) (at 113.97 83.82 0)
+    (effects (font (size 1.27 1.27)) (justify left)))
+  (global_label "UART_RX" (shape input) (at 113.97 86.36 0)
+    (effects (font (size 1.27 1.27)) (justify left)))
+  (wire (pts (xy 120.65 83.82) (xy 132.08 83.82)))
+  (wire (pts (xy 120.65 86.36) (xy 132.08 86.36)))
+  (wire (pts (xy 132.08 83.82) (xy 132.08 91.44)))
+  (wire (pts (xy 132.08 86.36) (xy 132.08 91.44)))
+  (wire (pts (xy 132.08 91.44) (xy 139.7 91.44)))
+  (global_label "GND" (shape passive) (at 139.7 91.44 0)
+    (effects (font (size 1.27 1.27)) (justify left)))
+  (global_label "UART_TX" (shape output) (at 86.36 81.28 180)
+    (effects (font (size 1.27 1.27)) (justify right)))
+  (global_label "UART_RX" (shape input) (at 86.36 83.82 180)
+    (effects (font (size 1.27 1.27)) (justify right)))
+  (global_label "BOOT0" (shape input) (at 50.8 152.4 0)
+    (effects (font (size 1.27 1.27)) (justify left)))
+  (wire (pts (xy 50.8 152.4) (xy 60.96 152.4)))
+  (wire (pts (xy 60.96 152.4) (xy 60.96 157.48)))
+  (global_label "GND" (shape passive) (at 60.96 157.48 270)
+    (effects (font (size 1.27 1.27)) (justify left)))
+  (wire (pts (xy 50.8 152.4) (xy 50.8 144.78)))
+  (global_label "+3V3" (shape passive) (at 50.8 142.24 270)
+    (effects (font (size 1.27 1.27)) (justify left)))
+  (global_label "NRST_BTN" (shape input) (at 72.39 152.4 0)
+    (effects (font (size 1.27 1.27)) (justify left)))
+  (wire (pts (xy 72.39 152.4) (xy 82.55 152.4)))
+  (wire (pts (xy 82.55 152.4) (xy 82.55 157.48)))
+  (global_label "GND" (shape passive) (at 82.55 157.48 270)
+    (effects (font (size 1.27 1.27)) (justify left)))
+  (global_label "NRST_BTN" (shape output) (at 86.36 88.9 180)
+    (effects (font (size 1.27 1.27)) (justify right)))
   (text "=== MCU: STM32G041K6U6 ===" (at 78.74 47.63 0)
     (effects (font (size 1.5 1.5) bold)))
@@
   (text "=== TRACK CONNECTORS ===" (at 218.44 84.96 0)
     (effects (font (size 1.5 1.5) bold)))
+  (text "=== SWD DEBUG / FLASH HEADER (J10) ===" (at 116.84 48.26 0)
+    (effects (font (size 1.5 1.5) bold)))
+  (text "Pin 1: SWDIO (PA13)  Pin 2: SWDCLK (PA14)\nPin 3: GND            Pin 4: +3.3V (optional)\n2.54mm 4-pin header. Match your ST-Link V2/V3 pinout." (at 116.84 50.8 0)
+    (effects (font (size 1.0 1.0)) (justify left)))
+  (text "=== UART DEBUG / BOOTLOADER (J11) ===" (at 116.84 78.74 0)
+    (effects (font (size 1.5 1.5) bold)))
+  (text "Pin 1: TX PA9  (-> RX of USB-UART adapter)\nPin 2: RX PA10 (-> TX of USB-UART adapter)\nPin 3: GND\n115200 8N1, 3.3V logic. Telemetry CSV at 100ms interval.\nAlso used by ROM bootloader (hold BOOT0 + press NRST)." (at 116.84 81.28 0)
+    (effects (font (size 1.0 1.0)) (justify left)))
+  (text "=== BOOT0 BUTTON (J12) ===" (at 33.02 138.43 0)
+    (effects (font (size 1.5 1.5) bold)))
+  (text "J12: momentary button PB8/BOOT0 to 3.3V\nHold J12 + press J13 NRST = ROM bootloader entry\nFlash via J11 UART: stm32flash -w aart_brake.bin /dev/ttyUSB0" (at 33.02 141.0 0)
+    (effects (font (size 1.0 1.0)) (justify left)))
+  (text "=== NRST BUTTON (J13) ===" (at 66.04 138.43 0)
+    (effects (font (size 1.5 1.5) bold)))
+  (text "J13: momentary button NRST to GND\nPress while holding J12 BOOT0 to enter bootloader.\nRelease J13 first, then release J12." (at 66.04 141.0 0)
+    (effects (font (size 1.0 1.0)) (justify left)))
   (text "SAFE DEFAULT:\nR2 (10k) on GD1 input pulls HIGH when MCU off\n=> Q1 ON => motor dead-shorted = safe" (at 121.92 55.88 0)
     (effects (font (size 1.0 1.0)) (justify left)))
   (text "Q1: N-ch low-side brake FET\nTIM3_CH1 INVERTED polarity\nCCR=0 => FET ON => dead short\nCCR=2720 => ~8ohm\nCCR=3199 => FET OFF" (at 185.42 82.55 0)
     (effects (font (size 1.0 1.0)) (justify left)))
-  (text "Q2: P-ch high-side keep-alive FET\nTIM3_CH2 normal polarity\nCCR=0 => FET OFF\nCCR=774 => ~3V injected" (at 185.42 120.65 0)
+  (text "Q2: P-ch high-side keep-alive FET\nTIM3_CH2 normal polarity\nCCR=0 => FET OFF\nCCR=400 => ~2V injected at 16V rail" (at 185.42 120.65 0)
     (effects (font (size 1.0 1.0)) (justify left)))
   (text "D4: MODE C ESSENTIAL\nBlocks reverse current into Q2\nwhen Q1 hard-brakes the track.\nOmit on mode A/B-only boards." (at 210.82 132.08 0)
     (effects (font (size 1.0 1.0)) (justify left)))
-  (text "POT MAPPING (all modes):\nCCW => min brake (~8 ohm)\nCW  => max brake (dead short)\nMode A: centre = dead short\n        CW past centre = antibrake 0-3V" (at 10.16 106.68 0)
+  (text "POT MAPPING (all modes):\nCCW => min brake (~8 ohm)\nCW  => max brake (dead short)\nMode A: centre = dead short\n        CW past centre = positive anti-brake 0-2V" (at 10.16 106.68 0)
     (effects (font (size 1.0 1.0)) (justify left)))
-  (text "COMPONENT LIST:\nU1  STM32G041K6U6  QFN-32\nU2  AMS1117-3.3    SOT-223\nGD1 UCC27524       SOT-23-5  (brake gate driver)\nGD2 UCC27524       SOT-23-5  (keep-alive gate driver)\nQ1  IRLB3034       D2PAK     (N-ch brake FET)\nQ2  IRF9Z34N       D2PAK     (P-ch keep-alive FET)\nD1  P6KE15A        SMB       (TVS rail clamp)\nD2  SS34           SMB       (Q1 catch diode)\nD3  SS34           SMB       (Q2 catch diode)\nD4  SS34           SMB       (mode C series protection)\nD5  LED Red        0805      (status LED)\nF1  Polyfuse 25A   1812\nC1  10uF  0805  C2  100nF 0402  (LDO in decouple)\nC3  10uF  0805  C4  100nF 0402  (LDO out decouple)\nC5  100nF 0402  C6  100nF 0402  C7  4u7 0402  (MCU decouple)\nR1  10k 0402 (NRST)  R2  10k 0402 (safe default)\nR3  10R 0402 (Q1 gate)  R4  10R 0402 (Q2 gate)\nR5  10k 0402 (pot ref)  R6  10k 0402 (btn pullup)\nR7  1k  0402 (btn series)  R8  15k 0402  R9  4k7 0402 (rail sense)\nR10 330R 0402 (LED)\nJ1  2-pin 5mm (track output)  J2  2-pin 5mm (12V rail in)\nJ3  2-pin 5mm (controller in)  J4  3-pin 2.54mm (pot)\nJ5  3-pin 2.54mm (toggle)  J6  2-pin 2.54mm (capture btn)\nJ7  2-pin 2.54mm (wiper strip)" (at 10.16 131.0 0)
+  (text "COMPONENT LIST (Rev 9):\nU1  STM32G041K6U6  QFN-32\nU2  AMS1117-3.3    SOT-223\nGD1 UCC27524       SOT-23-5  (brake gate driver)\nGD2 UCC27524       SOT-23-5  (keep-alive gate driver)\nQ1  IRLB3034       D2PAK     (N-ch brake FET)\nQ2  IRF9Z34N       D2PAK     (P-ch keep-alive FET)\nD1  P6KE18CA       SMB       (TVS BIDIRECTIONAL - CA suffix essential)\nD2  SS310          SMB       (Q1 catch - 100V required)\nD3  SS310          SMB       (Q2 catch - 100V required)\nD4  MBRS360/SS54   SMB       (mode C series - most stressed diode)\nD5  LED Red        0805      (status LED)\nF1  500mA-1A polyfuse  1812  (WHITE rail MCU supply ONLY)\nC1  10uF 0805  C2  100nF 0402  (LDO in)\nC3  10uF 0805  C4  100nF 0402  (LDO out)\nC5-C7  100nF/100nF/4u7 0402  (MCU decouple)\nR1  10k (NRST)  R2  10k (safe default on GD1 INPUT)\nR3  10R (Q1 gate)  R4  10R (Q2 gate)\nR5  10k (pot ref)  R6  10k (btn pullup)  R7  1k (btn series)\nR8  18k  R9  4k7  (WHITE sense)  R10  22k  R11  4k7  (BLACK sense)\nR12 330R (LED)\nJ1-J6   4mm banana sockets (track+ctrl WHITE/BLACK/RED)\nJ7  3-pin 2.54mm (mode toggle)\nJ8  2-pin 2.54mm (capture button)\nJ9  2-pin 4mm (track output)\nJ10 4-pin 2.54mm (SWD: SWDIO/SWDCLK/GND/+3V3)\nJ11 3-pin 2.54mm (UART: TX/RX/GND)\nJ12 2-pin 2.54mm (BOOT0 button)\nJ13 2-pin 2.54mm (NRST button)" (at 10.16 166.0 0)
+    (effects (font (size 1.0 1.0)) (justify left)))
+  (text "PLACEMENT GUIDE:\nTop-left:    Power (J1 rail, F1, D1, U2, C1-C4)\nTop-centre:  SWD J10 | UART J11\nLeft-mid:    Inputs (pot, toggle, capture btn, dividers)\nBelow-left:  BOOT0 J12 | NRST J13\nCentre:      MCU U1, C5-C7, R1\nRight-upper: Brake FET (GD1, R2, R3, Q1, D2)\nRight-lower: Keep-alive FET (GD2, R4, Q2, D3, D4)\nFar-right:   Track banana J1-J6\nBelow MCU:   Status LED R12 D5\nR2 pull-up: on GD1 INA input - NOT on Q1 gate" (at 10.16 210.0 0)
     (effects (font (size 1.0 1.0)) (justify left)))
 )

Commit message: Unwired KiCad
Other:
- added sheet 1 Power Supply (power_supply.kicad_sch)
- added sheet 2 MCU + Inputs (mcu_inputs.kicad_sch)
- added sheet 3 Debug + Flash Headers (debug_headers.kicad_sch)
- added sheet 4 Brake FET Circuit (brake_fet.kicad_sch)
- added sheet 5 Keep-alive FET Circuit (keepalive_fet.kicad_sch)
- added sheet 6 Track Connectors (track_connectors.kicad_sch)
- note added: "COMPONENT LIST (Rev 9):"
- note added: "Connectors J1-J6 4mm banana Track WHITE/BLACK/RED (x2 sides) J7 3-pin 2.54mm Mode toggle A/B/C J8 2-pin 2.54mm Capture button J9 2-pin 4mm Track output J10 4-pin 2.54mm SWD: SWDIO/SWDCLK/GND/+3V3 J11 3-pin 2.54mm UART: TX/RX/GND 115200 8N1 J12 2-pin 2.54mm BOOT0 button (ROM bootloader) J13 2-pin 2.54mm NRST button"
- note added: "FETs and Diodes Q1 IRLB3034 D2PAK N-ch brake FET (195A 40V) Q2 IRF9Z34N D2PAK P-ch keep-alive FET (18A 55V) D1 P6KE18CA SMB TVS bidirectional — CA suffix ESSENTIAL D2 SS310 SMB Q1 catch diode 100V required D3 SS310 SMB Q2 catch diode 100V required D4 MBRS360 SMB Mode C series protection — most stressed D5 LED Red 0805 Status LED"
- note added: "ICs U1 STM32G041K6U6 QFN-32 MCU U2 AMS1117-3.3 SOT-223 LDO 12-16V -> 3.3V GD1 UCC27524 SOT-23-5 Brake gate driver GD2 UCC27524 SOT-23-5 Keep-alive gate driver"
- note added: "KEY DESIGN NOTES:"
- note added: "Passives F1 500mA-1A polyfuse 1812 WHITE rail MCU supply ONLY C1 10uF 0805 LDO input bulk C2 100nF 0402 LDO input HF C3 10uF 0805 LDO output bulk C4 100nF 0402 LDO output HF C5 100nF 0402 MCU VDD decouple C6 100nF 0402 MCU VDDA decouple C7 4u7 0402 MCU VDDA bulk"
- note added: "Q1 TIM3_CH1 INVERTED polarity: CCR=0 = FET ON = dead short R2 pull-up on GD1 INPUT (not Q1 gate) = safe default brake at power-off D4 ESSENTIAL in mode C: blocks reverse current into Q2 during hard braking F1 in WHITE rail ONLY — never in BLACK track path (40A motor startup) D1 P6KE18CA — bidirectional variant — clamps both polarity transients D2/D3 SS310 100V — inductive turn-off spikes on 16V r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"
- note added: "Resistors R1 10k 0402 NRST pull-up R2 10k 0402 GD1 safe-default (on INPUT not gate) R3 10R 0402 Q1 gate R4 10R 0402 Q2 gate R5 10k 0402 Pot reference to 3.3V R6 10k 0402 Capture btn pull-up R7 1k 0402 Capture btn series R8 18k 0402 WHITE sense top divider R9 4k7 0402 WHITE sense bottom R10 22k 0402 BLACK sense top divider R11 4k7 0402 BLACK sense bottom R12 330R 0402 Status LED"
- note removed: "=== BOOT0 BUTTON (J12) ==="
- note removed: "=== BRAKE FET CIRCUIT ==="
- note removed: "=== INPUTS ==="
- note removed: "=== KEEP-ALIVE FET CIRCUIT ==="
- note removed: "=== MCU: STM32G041K6U6 ==="
- note removed: "=== NRST BUTTON (J13) ==="
- note removed: "=== SWD DEBUG / FLASH HEADER (J10) ==="
- note removed: "=== TRACK CONNECTORS ==="
- note removed: "=== UART DEBUG / BOOTLOADER (J11) ==="
- note removed: "COMPONENT LIST (Rev 9): U1 STM32G041K6U6 QFN-32 U2 AMS1117-3.3 SOT-223 GD1 UCC27524 SOT-23-5 (brake gate driver) GD2 UCC27524 SOT-23-5 (keep-alive gate driver) Q1 IRLB3034 D2PAK (N-ch brake FET) Q2 IRF9Z34N D2PAK (P-ch keep-alive FET) D1 P6KE18CA SMB (TVS BIDIRECTIONAL - CA suffix essential) D2 SS310 SMB (Q1 catch - 100V required) D3 SS310 SMB (Q2 catch - 100V required) D4 MBRS360/SS54 SMB (mode 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"
- note removed: "D4: MODE C ESSENTIAL Blocks reverse current into Q2 when Q1 hard-brakes the track. Omit on mode A/B-only boards."
- note removed: "J12: momentary button PB8/BOOT0 to 3.3V Hold J12 + press J13 NRST = ROM bootloader entry Flash via J11 UART: stm32flash -w aart_brake.bin /dev/ttyUSB0"
- note removed: "J13: momentary button NRST to GND Press while holding J12 BOOT0 to enter bootloader. Release J13 first, then release J12."
- note removed: "PLACEMENT GUIDE: Top-left: Power (J1 rail, F1, D1, U2, C1-C4) Top-centre: SWD J10 | UART J11 Left-mid: Inputs (pot, toggle, capture btn, dividers) Below-left: BOOT0 J12 | NRST J13 Centre: MCU U1, C5-C7, R1 Right-upper: Brake FET (GD1, R2, R3, Q1, D2) Right-lower: Keep-alive FET (GD2, R4, Q2, D3, D4) Far-right: Track banana J1-J6 Below MCU: Status LED R12 D5 R2 pull-up: on GD1 INA input - NOT on Q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"
- note removed: "POT MAPPING (all modes): CCW => min brake (~8 ohm) CW => max brake (dead short) Mode A: centre = dead short CW past centre = positive anti-brake 0-2V"
- note removed: "Pin 1: SWDIO (PA13) Pin 2: SWDCLK (PA14) Pin 3: GND Pin 4: +3.3V (optional) 2.54mm 4-pin header. Match your ST-Link V2/V3 pinout."
- note removed: "Pin 1: TX PA9 (-> RX of USB-UART adapter) Pin 2: RX PA10 (-> TX of USB-UART adapter) Pin 3: GND 115200 8N1, 3.3V logic. Telemetry CSV at 100ms interval. Also used by ROM bootloader (hold BOOT0 + press NRST)."
- note removed: "Q1: N-ch low-side brake FET TIM3_CH1 INVERTED polarity CCR=0 => FET ON => dead short CCR=2720 => ~8ohm CCR=3199 => FET OFF"
- note removed: "Q2: P-ch high-side keep-alive FET TIM3_CH2 normal polarity CCR=0 => FET OFF CCR=400 => ~2V injected at 16V rail"
- note removed: "SAFE DEFAULT: R2 (10k) on GD1 input pulls HIGH when MCU off => Q1 ON => motor dead-shorted = safe"
