File: aart-brake-kicad-h/aart_brake.kicad_sch (KiCad schematic)
At the start: 0 parts

Commit message: Update
Other:
- removed sheet 4 Brake FET Circuit
- removed sheet 5 Keep-alive FET Circuit
- added sheet 4 Brake FET (Q2 IRFP250N) (brake_fet.kicad_sch)
- added sheet 5 Anti-brake current src (Q1 TIP147) (keepalive_fet.kicad_sch)
- added sheet 7 Reverse-Block Switch (Q5/Q6 + TPS1212-Q1) (reverse_switch.kicad_sch)
- sheet 1 Power Supply ports: added +5V; removed none
- sheet 2 MCU + Inputs ports: added BLACK_SENSE, DAC1_Q2_BRAKE, KA_PWM_DEMAND, PB3_SW_EN, RAIL_SENSE; removed BLACK_SENSE_ADC, PA6_BRAKE_PWM, PA7_KA_PWM, SWDCLK, WHITE_SENSE_ADC
- sheet 3 Debug + Flash Headers ports: added none; removed SWDCLK
- sheet 6 Track Connectors ports: added CTRL_BLACK_IN; removed none
- note added: "- Reverse-block pass element = two N-ch (Q5/Q6, common-source) + U5 TPS1212-Q1 driven from WHITE (VS, not anode). RSNS current sense; I_DIR reverse (~6-10us) + I2t OCP + 5us SCP + IMON/FLT. Sits in BLACK CONTROLLER path. ~67-77mV at 40A (with RSNS). - BLACK sense (PA1) is on the TRACK side of the pass switch. - D1 TVS is on the WHITE rail only (transient clamp). - Anti-brake = constant-CURRENT so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"
- note added: "COMPONENT LIST (Revision 11):"
- note added: "Connectors J1-J6 4mm banana Track + controller WHITE/BLACK/RED (x2 sides) J7 3-pin 2.54mm Mode toggle A/B/C (PB0/PB1/GND) J10 4-pin SWD J11 3-pin UART J12 BOOT0 J13 NRST J14 3-pin voltmeter NOTE: J9 capture button REMOVED (toggle replaces it; PB3 reserved/optional)"
- note added: "FETs / power devices Q2 IRFP250N TO-247 Wide-SOA N-ch brake FET (30A 200V) + HEATSINK Q1 TIP147 TO-220 PNP Darlington anti-brake current-source pass (100V 10A 125W) + HEATSINK (alt: N-MOSFET SUP70060E / RFP50N06 / FDP61N20) Rsense 0.1ohm 1-2W anti-brake current sense (0.3V at 3A) Q_LS 2N2222 PWM level-shift C_KA 470n + R 10k/1k PWM->DC demand filter Q5 STL059N4S8AG PowerFLAT Reverse-block N-ch (4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"
- note added: "ICs U1 STM32G051K6U6 QFN-32 MCU (dual DAC, libopencm3, FW Rev 11) U2 AMS1117-3.3 / MCP1700 SOT-223/23 LDO 12-16V -> 3.3V (see 7A.6) U4 MCP1700-5002 SOT-23 LDO 12-16V -> 5V rail (GD2 brake buffer only; GD1 on WHITE) GD2 op-amp buffer SOT-23-5 Brake gate buffer (DAC1 -> Q2, linear) GD1 HV op-amp SOT-23-5 Anti-brake CURRENT-SOURCE loop on WHITE rail (PWM demand -> Q1; Rsense 0.1ohm) U5 TPS1212-Q1 VQ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"
- note added: "KEY DESIGN NOTES (Rev 11):"
- note added: "Passives F1 500mA-1A polyfuse 1812 WHITE rail MCU/analog supply ONLY (never BLACK) R2 10k 0402 GD2 input safe-default pull-up R3 10R 0402 Q2 gate R_BASE 1k 0402 Q1 Darlington base Rsense 0.1ohm anti-brake current sense RSNS ~0.5-0.75mohm TPS1212 main-path sense Q_LS 2N2222 PWM level-shift C_KA 470n + R 10k/1k PWM->DC filter R8 15k / R9 4k7 WHITE sense divider (PA0) R10 22k / R11 4k7 BLACK sense d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"
- note removed: "COMPONENT LIST (Rev 9):"
- note removed: "Connectors J1-J6 4mm banana Track WHITE/BLACK/RED (x2 sides) J7 3-pin 2.54mm Mode toggle A/B/C J8 2-pin 2.54mm Capture button J9 2-pin 4mm Track output J10 4-pin 2.54mm SWD: SWDIO/SWDCLK/GND/+3V3 J11 3-pin 2.54mm UART: TX/RX/GND 115200 8N1 J12 2-pin 2.54mm BOOT0 button (ROM bootloader) J13 2-pin 2.54mm NRST button J14 3-pin 2.54mm Voltmeter: Pin1=Vin(sig), Pin2=GND, Pin3=Vcc"
- note removed: "FETs and Diodes Q2 IRLB3034 D2PAK N-ch brake FET (195A 40V) Q1 IRF9Z34N D2PAK P-ch keep-alive FET (18A 55V) D1 P6KE18CA SMB TVS bidirectional — CA suffix ESSENTIAL D2 SS310 SMB Q2 catch diode 100V required D3 SS310 SMB Q1 catch diode 100V required D4 MBRS360 SMB Mode C series protection — most stressed D5 SS310 SMB Voltmeter isolation (D_V) — blocks PWM from WHITE rail D5 LED Red 0805 Status LED"
- note removed: "ICs U1 STM32G051K6U6 QFN-32 MCU U2 AMS1117-3.3 SOT-223 LDO 12-16V -> 3.3V GD2 UCC27524 SOT-23-5 Brake gate driver GD1 LM321 SOT-23-5 Q1 floating gate driver (WHITE-referenced supply) ZD1 BZX84C15 SOT-23 15V zener, GD1 floating supply (cathode=WHITE) U3 CH340N SOP-8 USB-UART bridge (JLCPCB C506813, no crystal needed) J_USB HRO TYPE-C-31-M-12 USB-C 16-pin receptacle D_USB BAT54 SOT-23 VBUS isolatio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"
- note removed: "KEY DESIGN NOTES: D_PG (pass gate) is in BLACK controller path, NOT WHITE rail. D1 TVS is on WHITE rail (transient clamp only). Black sense point (PA1) is on MOTOR SIDE of D_PG."
- note removed: "Passives F1 500mA-1A polyfuse 1812 WHITE rail MCU supply ONLY C1 10uF 0805 LDO input bulk C2 100nF 0402 LDO input HF C3 10uF 0805 LDO output bulk C4 100nF 0402 LDO output HF C5 100nF 0402 MCU VDD decouple C6 100nF 0402 MCU VDDA decouple C7 4u7 0402 MCU VDDA bulk C_VM 100uF SMD Voltmeter RC filter cap (with R_VM 10k, tau=1s)"
- note removed: "Q2 TIM3_CH1 INVERTED polarity: CCR=0 = FET ON = dead short R2 pull-up on GD2 INPUT (not Q2 gate) = safe default brake at power-off D4 ESSENTIAL in mode C: blocks reverse current into Q1 during hard braking F1 in WHITE rail ONLY — never in BLACK track path (40A motor startup) D1 P6KE18CA — bidirectional variant — clamps both polarity transients D2/D3 SS310 100V — inductive turn-off spikes on 16V r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"
- note removed: "Resistors R1 10k 0402 NRST pull-up R2 10k 0402 GD2 safe-default (on INPUT not gate) R3 10R 0402 Q2 gate R4 10R 0402 Q1 gate R5 10k 0402 Pot reference to 3.3V R6 10k 0402 Capture btn pull-up R7 1k 0402 Capture btn series R8 18k 0402 WHITE sense top divider R9 4k7 0402 WHITE sense bottom R10 22k 0402 BLACK sense top divider R11 4k7 0402 BLACK sense bottom R12 330R 0402 Status LED R_W 10k 0402 Voltm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"
