File: aart-brake-kicad-h/aart_brake.kicad_sch (KiCad schematic)
At the start: 0 parts

Commit message: Latest
Other:
- removed sheet 4 Brake FET (Q2 IRFP250N)
- removed sheet 7 Reverse-Block Switch (Q5/Q6 + TPS1212-Q1)
- added sheet 4 Brake FET (Q2 TW100N03CC) (brake_fet.kicad_sch)
- added sheet 7 Reverse-Block Switch (Q5/Q6 + INA210/LM311 ideal diode) (reverse_switch.kicad_sch)
- sheet 2 MCU + Inputs ports: added KA_DAC_DEMAND; removed KA_PWM_DEMAND
- sheet 5 Anti-brake current src (Q1 TIP147) ports: added KA_DAC_DEMAND; removed KA_PWM_DEMAND
- note added: "- Reverse-block pass element = two N-ch (Q5/Q6, common-source) + INA210/LM311 ideal diode INA210 (gain 200, +5V) across Rsns_sw; LM311 (~50mV hyst) trips on reverse (~0.16A, ~2us) -> gate driver off + PA6 brake-detect. No I2t/SCP/IMON (open items); gate-drive charge pump from WHITE to lift gates above BLACK (open item). Sits in BLACK CONTROLLER path. ~87mV at 40A. - BLACK sense (PA1) is on the TR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"
- note added: "Connectors J1-J6 4mm banana Track + controller WHITE/BLACK/RED (x2 sides) J7 3-pin 2.54mm Mode toggle A/B/C (PB0/PB1/GND) J10 4-pin SWD J11 3-pin UART J12 BOOT0 J13 NRST J14 4-pin TM1637 display (CLK/DIO/GND/VCC) NOTE: J9 capture button REMOVED (toggle replaces it; PB3 reserved/optional)"
- note added: "FETs / power devices Q2 TW100N03CC D2PAK Low-Rds logic-level N-ch brake FET (~3mohm 30V); IRFP250N=brushed-only alt Q1 TIP147 TO-220 PNP Darlington anti-brake current-source pass (100V 10A 125W) + HEATSINK (alt: N-MOSFET SUP70060E / RFP50N06 / FDP61N20) Rsense 0.1ohm 1-2W anti-brake current sense (0.3V at 3A) R_KA1 6.8k/R_KA2 1.2k DAC2 anti-brake divider GD3 LM7321 DAC2->WHITE level translator Q5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"
- note added: "ICs U1 STM32G051K6U6 QFN-32 MCU (dual DAC, libopencm3, FW Rev 11) U2 AMS1117-3.3 / MCP1700 SOT-223/23 LDO 12-16V -> 3.3V (see 7A.6) U4 MCP1700-5002 SOT-23 LDO 12-16V -> 5V rail (GD2 brake buffer only; GD1 on WHITE) GD2 op-amp buffer SOT-23-5 Brake gate buffer (DAC1 -> Q2, linear) GD1 HV op-amp SOT-23-5 Anti-brake CURRENT-SOURCE loop on WHITE rail (PWM demand -> Q1; Rsense 0.1ohm) U5 INA210 SC70-6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"
- note added: "Passives F1 500mA-1A polyfuse 1812 WHITE rail MCU/analog supply ONLY (never BLACK) R2 10k 0402 GD2 input safe-default pull-up R3 10R 0402 Q2 gate R_BASE 1k 0402 Q1 Darlington base Rsense 0.1ohm anti-brake current sense Rsns_sw ~1mohm ideal-diode shunt R_KA1 6.8k/R_KA2 1.2k DAC2 anti-brake divider (feeds GD3 LM7321 translator) R8 15k / R9 4k7 WHITE sense divider (PA0) R10 22k / R11 4k7 BLACK sense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"
- note removed: "- Reverse-block pass element = two N-ch (Q5/Q6, common-source) + U5 TPS1212-Q1 driven from WHITE (VS, not anode). RSNS current sense; I_DIR reverse (~6-10us) + I2t OCP + 5us SCP + IMON/FLT. Sits in BLACK CONTROLLER path. ~67-77mV at 40A (with RSNS). - BLACK sense (PA1) is on the TRACK side of the pass switch. - D1 TVS is on the WHITE rail only (transient clamp). - Anti-brake = constant-CURRENT so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"
- note removed: "Connectors J1-J6 4mm banana Track + controller WHITE/BLACK/RED (x2 sides) J7 3-pin 2.54mm Mode toggle A/B/C (PB0/PB1/GND) J10 4-pin SWD J11 3-pin UART J12 BOOT0 J13 NRST J14 3-pin voltmeter NOTE: J9 capture button REMOVED (toggle replaces it; PB3 reserved/optional)"
- note removed: "FETs / power devices Q2 IRFP250N TO-247 Wide-SOA N-ch brake FET (30A 200V) + HEATSINK Q1 TIP147 TO-220 PNP Darlington anti-brake current-source pass (100V 10A 125W) + HEATSINK (alt: N-MOSFET SUP70060E / RFP50N06 / FDP61N20) Rsense 0.1ohm 1-2W anti-brake current sense (0.3V at 3A) Q_LS 2N2222 PWM level-shift C_KA 470n + R 10k/1k PWM->DC demand filter Q5 STL059N4S8AG PowerFLAT Reverse-block N-ch (4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"
- note removed: "ICs U1 STM32G051K6U6 QFN-32 MCU (dual DAC, libopencm3, FW Rev 11) U2 AMS1117-3.3 / MCP1700 SOT-223/23 LDO 12-16V -> 3.3V (see 7A.6) U4 MCP1700-5002 SOT-23 LDO 12-16V -> 5V rail (GD2 brake buffer only; GD1 on WHITE) GD2 op-amp buffer SOT-23-5 Brake gate buffer (DAC1 -> Q2, linear) GD1 HV op-amp SOT-23-5 Anti-brake CURRENT-SOURCE loop on WHITE rail (PWM demand -> Q1; Rsense 0.1ohm) U5 TPS1212-Q1 VQ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"
- note removed: "Passives F1 500mA-1A polyfuse 1812 WHITE rail MCU/analog supply ONLY (never BLACK) R2 10k 0402 GD2 input safe-default pull-up R3 10R 0402 Q2 gate R_BASE 1k 0402 Q1 Darlington base Rsense 0.1ohm anti-brake current sense RSNS ~0.5-0.75mohm TPS1212 main-path sense Q_LS 2N2222 PWM level-shift C_KA 470n + R 10k/1k PWM->DC filter R8 15k / R9 4k7 WHITE sense divider (PA0) R10 22k / R11 4k7 BLACK sense d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"
