File: aart-brake-kicad-h/brake_fet.kicad_sch (KiCad schematic)
At the start: 0 parts

Commit message: Update
Other:
- note added: "D2 SS310 CATCH DIODE — ESSENTIAL: Motor inductance produces a large voltage spike on current interruption. SS310 (100V) chosen for headroom on the 16V rail. Clamps the spike to Vf + Vdc."
- note added: "GD2 op-amp buffer (+5V rail) SOT-23-5"
- note added: "Q2 IRFP250N wide-SOA N-ch TO-247 + heatsink 30A 200V"
- note added: "Q2 IRFP250N — WIDE-SOA, HEATSINK REQUIRED: Linear operation requires a wide-SOA planar part. The former IRLB3034 (trench switching FET) has poor linear-mode SOA and risks secondary breakdown. Worst-case ~12W mid-range; brake is intermittent (~10-20% duty) but the heatsink must take the peak. See design doc 7A.8.1."
- note added: "RESISTANCE-CONTROLLED BRAKE (linear, no PWM): DAC1 (0-3.3V) -> GD2 op-amp buffer -> Q2 gate. Q2 is operated in its LINEAR region: gate voltage sets Rds, which is placed across the motor (low-side, TRACK_POS to RED). Mode B indexes one of seven stored brake tables (25/15/5/4/3/2/1 ohm full scale); Mode A linear-maps the pot. No switching, no PWM, no switching noise."
- note added: "SAFE DEFAULT — CRITICAL: R2 (10k) is on the GD2 INPUT pin, NOT on Q2 gate. When the MCU is unpowered/reset, the GD2 input is pulled to a safe-default level so Q2 defaults to braking. If R2 were on the gate, the buffer would fight it."
- note removed: "D2 SS310 CATCH DIODE — ESSENTIAL: Motor inductance produces a large voltage spike on Q2 turn-off. Unclamped: L x dI/dt = 100uH x 20A/1us = 2000V Q2 Vds(max) = 40V — would be instantly destroyed. D2 clamps the spike at Vf + Vdc ~= 12.5V, absorbing ~20mJ. SS310 (100V) chosen over SS34 (40V) for headroom on 16V rail."
- note removed: "GD2 UCC27524 SOT-23-5"
- note removed: "INVERTED POLARITY — WHY: TIM3_CH1 is configured with inverted output polarity. CCR = 0 => output pin HIGH => Q2 ON => dead short CCR = 2720 => PWM ~85% HIGH => ~8ohm effective CCR = 3199(ARR) => output pin LOW => Q2 OFF This is the opposite of the normal PWM convention but guarantees the safe state at CCR=0 and at power-off."
- note removed: "Q2 IRLB3034 N-ch D2PAK 195A 40V"
- note removed: "SAFE DEFAULT — CRITICAL: R2 (10k) is on GD2 input pin, NOT on Q2 gate. When MCU is unpowered/reset, GD2 input floats HIGH via R2. GD2 drives Q2 gate HIGH => Q2 fully on => motor dead-shorted. This is the intended safe failure mode. If R2 were on Q2 gate, the gate driver would fight it."
