File: aart-brake-kicad-h/brake_fet.kicad_sch (KiCad schematic)
At the start: 0 parts

Commit message: Latest
Other:
- note added: "GD2 RRO op-amp, +5V gain ~1.5 (3.3V DAC -> ~5V gate) e.g. TI LM7321 (RRO)"
- note added: "Q2 BRAKE FET — LOW-Rds, brushless-dominant (80%): Brushless braking shorts the Remora ESC bus; motor 31-273mohm is BELOW the FET Rds, so the brake is FET-limited. Q2 must be single- digit-mohm logic-level (e.g. TW100N03CC), driven FULL-ON. IRFP250N (75mohm) gives only 9-78% brake + ~120W at 40A => brushed-only. Brushed linear tables: low-Rds FET VALIDATED in linear - brushed op point is low Vds (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"
- note added: "Q2 low-Rds logic-level N-ch ~3mohm e.g. TW100N03CC FULL-ON for brushless IRFP250N = brushed-only"
- note added: "RESISTANCE-CONTROLLED BRAKE (linear, no PWM): DAC1 (0-3.3V) -> GD2 (non-inverting, gain ~1.5) -> ~5V max -> Q2 gate. Q2 is operated in its LINEAR region: gate voltage sets Rds, which is placed across the motor (low-side, TRACK_POS to RED). Mode B indexes one of seven stored brake tables (25/15/5/4/3/2/1 ohm full scale); Mode A linear-maps the pot. No switching, no PWM, no switching noise."
- note removed: "GD2 op-amp buffer (+5V rail) SOT-23-5"
- note removed: "Q2 IRFP250N wide-SOA N-ch TO-247 + heatsink 30A 200V"
- note removed: "Q2 IRFP250N — WIDE-SOA, HEATSINK REQUIRED: Linear operation requires a wide-SOA planar part. The former IRLB3034 (trench switching FET) has poor linear-mode SOA and risks secondary breakdown. Worst-case ~12W mid-range; brake is intermittent (~10-20% duty) but the heatsink must take the peak. See design doc 7A.8.1."
- note removed: "RESISTANCE-CONTROLLED BRAKE (linear, no PWM): DAC1 (0-3.3V) -> GD2 op-amp buffer -> Q2 gate. Q2 is operated in its LINEAR region: gate voltage sets Rds, which is placed across the motor (low-side, TRACK_POS to RED). Mode B indexes one of seven stored brake tables (25/15/5/4/3/2/1 ohm full scale); Mode A linear-maps the pot. No switching, no PWM, no switching noise."
