File: aart-brake-kicad-h/keepalive_fet.kicad_sch (KiCad schematic)
At the start: 0 parts

Commit message: Update
Other:
- note added: "ANTI-BRAKE = CONSTANT-CURRENT SOURCE (this revision): Classic high-side op-amp current source. GD1 drives Q1 and regulates the drop across Rsense (0.1 ohm) to equal the demand, holding I = Vdemand/Rsense regardless of motor. Demand: a 50kHz MCU PWM, level-shifted (2N2222) and RC-filtered (470n + R) to 0-0.3V. Pot sets PWM duty -> current. 0% = 0A (off); full = 3A. Why a current source: a stalled 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"
- note added: "D4 MBRS360 reverse block"
- note added: "GD1 HV op-amp current loop (WHITE rail, 0-16V) LM321/LM358-class >=16V"
- note added: "OP-AMP SUPPLY - CRITICAL: GD1 is powered from the WHITE rail (~16V), NOT +5V. Rsense is in the WHITE leg, so the op-amp inputs/output sit at ~16V common mode; a 5V op-amp cannot work here. Use a single-supply HV op-amp (LM321/LM358-class, >=16V, ideally 36V), GND-to-WHITE. Confirmed by the SIMetrix design (op-amp V+ = supply rail). Only GD2 (brake) is on +5V."
- note added: "Q1 TIP147 PNP Darlington TO-220 + heatsink (or N-MOSFET alt: SUP70060E/RFP50N06)"
- note added: "RETIRED - do NOT fit: floating-supply P-ch (ZD1/R_Z1/C_Z1/LM321, IRF9Z34N) and the voltage-follower TIP122 NPN. See design doc 7A.7."
- note added: "Rsense 0.1 ohm (WHITE leg) 0.3V at 3A"
- note added: "SAFETY: Shoot-through protection - if brake (Q2) and anti-brake fault on together, the current source caps its contribution at ~3A instead of feeding a near-short. Add open/short detection on the loop + fast OCP to guard source component failure."
- note added: "THERMAL (steady-state baseline, from SIMetrix design): Vsupply max 16V, Ta 30C. At 2.75A -> Pd 44W (47W at full 3A). TIP147: SOA 125W@25C, Tj allow 125C, Rthjc 1C/W -> Rthca 1.16C/W, Tc 81C. SUP70060E: SOA 200W, Tj 150C, Rthjc 0.75 -> Rthca 1.98C/W, Tc 117C (smaller sink, hotter). Anti-brake is bursty: size heatsink by pulse energy / thermal capacitance (dT ~= Energy/Cth) not steady 47W - a ~50g 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"
- note added: "level shift + PWM->DC filter 2N2222 + 470n + 10k/1k (KA_PWM_DEMAND from MCU 50kHz)"
- note removed: "D3 SS310 CATCH DIODE: Connected across Q1 drain-source. Protects against inductive voltage spikes on Q1 turn-off. 100V rating required on 16V rail — same reasoning as D2."
- note removed: "D3 SS310 catch 100V"
- note removed: "D4 MBRS360 series output"
- note removed: "D4 MBRS360 — MODE C ESSENTIAL: In mode C, Q1 injects keep-alive while Q2 may simultaneously deadshort the track. D4 blocks reverse current back through Q1. Without D4: Q1 body diode conducts ~46A at 20kHz repetitively. IRF9Z34N body diode is not rated for this. D4 is the most electrically stressed diode in this design. SS34 (3A/80A peak) is marginal. MBRS360 (3A/60V) is specified. D4 can be omitt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"
- note removed: "FLOATING SUPPLY CIRCUIT: ZD1 BZX84C15 (SOT-23) Cathode -> WHITE rail Anode -> GD1 V+ pin R_Z1 10k 0402 WHITE -> ZD1 cathode (current limit) C_Z1 100nF 0402 Across GD1 supply (ZD1 anode to GD1 V-) GD1 V- connected to WHITE-15V node (ZD1 anode). GD1 V+ connected to WHITE rail. Do NOT connect GD1 V- to GND."
- note removed: "GD1 UCC27524 SOT-23-5"
- note removed: "Q1 IRF9Z34N P-ch D2PAK 18A 55V"
- note removed: "Q1 P-CHANNEL GATE DRIVE (floating supply): GD1 (LM321) powered by floating supply: V+ = WHITE, V- = WHITE - 15V (via ZD1 + R_Z1). DAC2 (0-3.3V GND-ref) drives GD1 non-inverting input. GD1 output range: (WHITE-15V) to WHITE. DAC=4095 (3.3V) -> GD1 output -> WHITE -> Vgs=0V -> Q1 OFF (correct). DAC=2480 (~2V) -> GD1 output -> WHITE-13V -> Vgs=-13V -> Q1 max conduction. DAC=0 (0V) -> GD1 output -> W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"
- note removed: "R4 10R gate"
- note removed: "TIM3_CH2 NORMAL POLARITY: CCR = 0 => output pin LOW => Vgs negative => Q1 OFF CCR = 400(KA_MAX) => PWM 12.5% duty => ~2V effective at 16V rail Effective voltage = (CCR / 3200) x V_RAIL Adjust KA_MAX via UART: SET KA_MAX <ccr>"
- title: AART Brake Module — 5: Keep-alive FET Circuit -> AART Brake Module — 5: Anti-brake constant-current source (3A, PWM-set)
