File: aart-brake-kicad-h/keepalive_fet.kicad_sch (KiCad schematic)
At the start: 0 parts

Commit message: Latest
Other:
- note added: "ANTI-BRAKE = CONSTANT-CURRENT SOURCE (this revision): Classic high-side op-amp current source. GD1 drives Q1 and regulates the drop across Rsense (0.1 ohm) to equal the demand, holding I = Vdemand/Rsense regardless of motor. Demand: MCU DAC2 DC, scaled by R_KA1/R_KA2 divider + GD3 (LM7321) to 0-0.3V referred to WHITE. Pot sets DAC code -> current. code 0 = 0A (off); full = 3A. Why a current sourc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"
- note added: "DAC2 level translator R_KA1 6.8k/R_KA2 1.2k + GD3 LM7321 (KA_DAC_DEMAND from MCU DAC2 DC)"
- note added: "GD1 RRIO op-amp on WHITE rail (0-16V, input CMR must reach V+) e.g. TI LM7321 (RRIO, 2.5-32V)"
- note added: "OP-AMP SUPPLY - CRITICAL: GD1 is powered from the WHITE rail (~16V), NOT +5V. Rsense is in the WHITE leg, so the op-amp inputs/output sit at ~16V common mode; a 5V op-amp cannot work here. Use a RAIL-TO-RAIL INPUT op-amp whose input CMR includes V+ (e.g. TI LM7321, SOT-23, 2.5-32V RRIO). Ordinary LM358/LM321/LM324 stop ~1.5V below V+ and will NOT work here. Confirmed by the SIMetrix design (op-am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"
- note added: "RETIRED - do NOT fit: floating-supply P-ch (ZD1/R_Z1/C_Z1/LM321, IRF9Z34N) and the voltage-follower TIP122 NPN; 2N2222 PWM level-shift + C_KA RC filter (now DAC2 + GD3). See design doc 7A.7."
- note removed: "ANTI-BRAKE = CONSTANT-CURRENT SOURCE (this revision): Classic high-side op-amp current source. GD1 drives Q1 and regulates the drop across Rsense (0.1 ohm) to equal the demand, holding I = Vdemand/Rsense regardless of motor. Demand: a 50kHz MCU PWM, level-shifted (2N2222) and RC-filtered (470n + R) to 0-0.3V. Pot sets PWM duty -> current. 0% = 0A (off); full = 3A. Why a current source: a stalled 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"
- note removed: "GD1 HV op-amp current loop (WHITE rail, 0-16V) LM321/LM358-class >=16V"
- note removed: "OP-AMP SUPPLY - CRITICAL: GD1 is powered from the WHITE rail (~16V), NOT +5V. Rsense is in the WHITE leg, so the op-amp inputs/output sit at ~16V common mode; a 5V op-amp cannot work here. Use a single-supply HV op-amp (LM321/LM358-class, >=16V, ideally 36V), GND-to-WHITE. Confirmed by the SIMetrix design (op-amp V+ = supply rail). Only GD2 (brake) is on +5V."
- note removed: "RETIRED - do NOT fit: floating-supply P-ch (ZD1/R_Z1/C_Z1/LM321, IRF9Z34N) and the voltage-follower TIP122 NPN. See design doc 7A.7."
- note removed: "level shift + PWM->DC filter 2N2222 + 470n + 10k/1k (KA_PWM_DEMAND from MCU 50kHz)"
- title: AART Brake Module — 5: Anti-brake constant-current source (3A, PWM-set) -> AART Brake Module — 5: Anti-brake constant-current source (3A, DAC2-set)
