File: aart-brake-kicad-h/mcu_inputs.kicad_sch (KiCad schematic)
At the start: 0 parts

Commit message: Update
Other:
- note added: "DUAL DAC (replaces TIM3 PWM gate drive): PA4 DAC_CH1 and PA5 DAC_CH2 drive op-amp buffers in LINEAR mode (no switching, no EMI). DAC2 polarity is now non-inverted: 0% duty = off, full = 3A current source. PWM filtered to DC demand. See doc 7A.7/11.1."
- note added: "LEFT SIDE INPUTS:"
- note added: "PA0 ADC_IN0 WHITE rail sense R8=15k/R9=4k7 divider PA1 ADC_IN1 BLACK track sense R10=22k/R11=4k7 divider (track side of pass switch) PA3 ADC_IN3 Pot wiper (10k, CCW = min brake) PB0 GPIO in Toggle bit0 (mode select), pull-up, active-LOW PB1 GPIO in Toggle bit1 (mode select), pull-up, active-LOW PB3 GPIO Reserved (optional reverse-switch enable; unused in Rev 11)"
- note added: "PA4 DAC_CH1 Brake -> GD2 op-amp buffer -> Q2 (linear, no PWM) PA5 TIM PWM Anti-brake demand 50kHz -> level-shift+filter -> GD1 current source PB4 TIM3_CH1 Voltmeter PWM -> 10k/100uF RC -> D_V -> J14 PA9 USART1_TX UART debug/bootloader 115200 8N1 PA10 USART1_RX UART RX PA13 SWDIO SWD PA14 SWDCLK SWD PB6 GPIO out Status LED (blinks 3x on flash save) NRST Reset input"
- note added: "RAIL SENSE DIVIDERS: WHITE: R8=15k / R9=4k7 -> within 3.3V ADC at 16V rail BLACK: R10=22k / R11=4k7, tapped on the TRACK side of the pass switch"
- note added: "RIGHT SIDE OUTPUTS:"
- note added: "TOGGLE DECODING (PB0=bit0, PB1=bit1, active-LOW pull-up): PB0=H PB1=H -> Mode A (brake only, all motors; pot linear) PB0=L PB1=H -> Mode B (brake + anti-brake, brushed; coupled tables) PB0=H PB1=L -> Mode C (keep-alive tuning, brushless setup) both LOW -> defaults to Mode A"
- note removed: "LEFT SIDE INPUTS (PA0-PA5):"
- note removed: "PA0 ADC_IN0 WHITE rail sense R8=18k/R9=4k7 divider 3.31V at 16V PA1 ADC_IN1 BLACK track sense R10=22k/R11=4k7 divider 2.82V at 16V PA2 GPIO in Toggle bit0 (mode select) pull-up active-LOW PA3 ADC_IN3 Pot wiper (10k centre-detent, CCW=min brake) PA4 GPIO in Toggle bit1 (mode select) pull-up active-LOW PA5 ADC_IN5 Capture button (10k pull-up + 1k series to GND)"
- note removed: "PA6 TIM3_CH1 AF1 Brake PWM -> GD2 -> Q2 (INVERTED polarity) PA7 TIM3_CH2 AF1 Keep-alive PWM -> GD1 -> Q1 (normal polarity) PB4 TIM3_CH1 AF1 Voltmeter PWM -> 10k/100uF RC -> D_V -> J14 pin1 PA9 USART1_TX AF1 UART debug/bootloader TX 115200 8N1 PA10 USART1_RX AF1 UART RX PA13 SWDIO AF0 SWD debug interface PA14 SWDCLK AF0 SWD debug interface PB6 GPIO out Status LED (blinks 3x on flash save) NRST Res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"
- note removed: "RAIL SENSE DIVIDERS: WHITE: R8=18k (top) R9=4k7 (bot) -> 3.31V at 16V rail BLACK: R10=22k (top) R11=4k7 (bot) -> 2.82V at 16V rail Both safe for 3.3V ADC reference."
- note removed: "RIGHT SIDE OUTPUTS (PA6, PA7, PA9, PA10, PA13, PA14, PB6):"
- note removed: "TOGGLE DECODING: PA2=H PA4=H -> Mode A (brushed + positive anti-brake) PA2=L PA4=H -> Mode B (brushed, reduced braking only) PA2=H PA4=L -> Mode C (brushless, eCom keep-alive) PA2=L PA4=L -> invalid -> defaults to Mode B (safe)"
