File: aart-brake-kicad-h/mcu_inputs.kicad_sch (KiCad schematic)
At the start: 0 parts

Commit message: Latest
Other:
- note added: "DUAL DAC (replaces TIM3 PWM gate drive): PA4 DAC_CH1 and PA5 DAC_CH2 drive op-amp buffers in LINEAR mode (no switching, no EMI). DAC2 polarity is now non-inverted: code 0 = off, full = 3A current source. DAC output is DC; no PWM or RC filter. See doc 7A.7/11.1."
- note added: "PA4 DAC_CH1 Brake -> GD2 op-amp buffer -> Q2 (linear, no PWM) PA5 DAC_CH2 Anti-brake demand DC -> R_KA1/R_KA2 div -> GD3 LM7321 -> GD1 current source PB4 GPIO TM1637 display CLK -> J14 PA9 USART1_TX UART debug/bootloader 115200 8N1 PA10 USART1_RX UART RX PA13 SWDIO SWD PA14 SWDCLK SWD + BOOT0 (J12 via series R, nBOOT_SEL=0) PB6 GPIO out Status LED (blinks 3x on flash save) PB8 GPIO TM1637 display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"
- note removed: "DUAL DAC (replaces TIM3 PWM gate drive): PA4 DAC_CH1 and PA5 DAC_CH2 drive op-amp buffers in LINEAR mode (no switching, no EMI). DAC2 polarity is now non-inverted: 0% duty = off, full = 3A current source. PWM filtered to DC demand. See doc 7A.7/11.1."
- note removed: "PA4 DAC_CH1 Brake -> GD2 op-amp buffer -> Q2 (linear, no PWM) PA5 TIM PWM Anti-brake demand 50kHz -> level-shift+filter -> GD1 current source PB4 TIM3_CH1 Voltmeter PWM -> 10k/100uF RC -> D_V -> J14 PA9 USART1_TX UART debug/bootloader 115200 8N1 PA10 USART1_RX UART RX PA13 SWDIO SWD PA14 SWDCLK SWD PB6 GPIO out Status LED (blinks 3x on flash save) NRST Reset input"
