File: aart-brake-kicad-h/power_supply.kicad_sch (KiCad schematic)
At the start: 0 parts

Commit message: Update
Other:
- note added: "+3V3 RAIL (U2): 16.0V rail: P = (16.0-3.3) x 0.035 = 0.44W, dT ~27C in SOT-223. AMS1117 handles the thermal at 16V in but has ~5mA quiescent; MCP1700 is 2uA Iq but higher Rth in SOT-23 — pick per standby budget vs package thermal (see design doc 7A.6)."
- note added: "+5V RAIL (U4): Feeds the GD2 brake-buffer op-amp only. NOTE: the GD1 anti-brake current-source op-amp is NOT on this rail - it is powered from WHITE (~16V) because it senses in the WHITE leg at ~16V common mode (a 5V op-amp cannot). ~11V drop from WHITE at mA-level load = negligible heat in SOT-23."
- note added: "C1 C2 LDO in"
- note added: "D1 P6KE18CA TVS bidir"
- note added: "J2 WHITE"
- note added: "TPS1212-Q1 SUPPLY (no clamp): The reverse-switch controller U5 (TPS1212-Q1) VS pin connects to WHITE directly - its 3.5-73V range covers the 16V rail, so the DZ1/RZ1 zener clamp the LTC7001 needed is removed. U5 also self-protects via I2t/SCP. See reverse_switch sheet."
- note added: "TVS selection: P6KE18CA bidirectional (CA suffix) ESSENTIAL — clamps both polarities of inductive transient on the WHITE rail."
- note added: "U2 AMS1117-3.3 (or MCP1700) SOT-223 -> +3V3"
- note added: "U4 MCP1700-5002 SOT-23 -> +5V analog rail"
- note added: "USB POWER PATH: VBUS -> F_USB (500mA polyfuse) -> D_USB (BAT54) -> LDO input node. D_USB anode=VBUS, cathode=LDO_in. Reversed = HOST DAMAGE. R_CC1/R_CC2 5.1k CC pull-downs; C_USB1 10uF VBUS bulk."
- note removed: "4mm banana WHITE input +12-16V always-live from track PSU (40-90A source) Module draws only ~35mA from this rail via F1 and LDO Track power path (BLACK) bypasses this circuit entirely"
- note removed: "C1 C2 LDO in decouple"
- note removed: "C3 C4 LDO out decouple"
- note removed: "D1 P6KE18CA TVS bidirectional"
- note removed: "J2"
- note removed: "LDO power dissipation: 12.4V rail: P = (12.4-3.3) x 0.035 = 0.32W, dT = 20C 16.0V rail: P = (16.0-3.3) x 0.035 = 0.44W, dT = 27C Both within AMS1117-3.3 125C Tj limit at 25C ambient. Solder SOT-223 tab to copper pour for best performance."
- note removed: "TVS selection note: P6KE18CA — bidirectional (CA suffix) is ESSENTIAL. Unidirectional P6KE18A only clamps one polarity. Inductive switching on this rail produces transients in both directions."
- note removed: "U2 AMS1117-3.3 SOT-223"
- note removed: "USB POWER PATH: VBUS -> F_USB (500mA polyfuse) -> D_USB (BAT54, SOT-23) -> LDO input node (joins WHITE path after D_WHITE) D_USB: anode=VBUS_fused, cathode=LDO_input D_USB CRITICAL: must be oriented correctly. Reversed D_USB = track voltage on USB host = HOST DAMAGE. C_USB1: 10uF 10V MLCC 0805 on VBUS (before F_USB) F_USB: 500mA polyfuse 0805 R_CC1: 5.1k 0402, CC1->GND R_CC2: 5.1k 0402, CC2->GND"
