File: aart-brake-kicad-h/power_supply.kicad_sch (KiCad schematic)
At the start: 0 parts

Commit message: Latest
Other:
- note added: "IDEAL-DIODE SUPPLY: The reverse-switch sense amp U5 (INA210) and comparator U6 (LM311) run off the +5V LDO rail. The Q5/Q6 common-source gates need a high-side gate driver / charge pump fed from WHITE (open item). No self-protection (I2t/SCP). See reverse_switch sheet."
- note removed: "TPS1212-Q1 SUPPLY (no clamp): The reverse-switch controller U5 (TPS1212-Q1) VS pin connects to WHITE directly - its 3.5-73V range covers the 16V rail, so the DZ1/RZ1 zener clamp the LTC7001 needed is removed. U5 also self-protects via I2t/SCP. See reverse_switch sheet."
