File: aart-brake-kicad-h/track_connectors.kicad_sch (KiCad schematic)
At the start: 0 parts

Commit message: Update
Other:
- note added: "BLACK PATH IS BROKEN HERE BY THE REVERSE SWITCH: Track BLACK (J3) = TRACK_POS. Controller BLACK (J4) = CTRL_BLACK_IN. These are SEPARATE nets — the two N-ch reverse-block switch (sheet 7) sits between them. WHITE (J1/J2 = +12V_RAIL) and RED (J5/J6 = GND) pass straight through; only BLACK is switched."
- note added: "BRAKE DETECTION (this module): V_BLACK < 500mV => enter brake state V_BLACK > 1500mV => exit brake state Hysteresis prevents chatter at low throttle."
- note added: "Module inserts between track and controller. During normal forward drive the switch is fully on (low Rds), so the module is near-transparent on BLACK (~27-47mV at 40A). Brake detection: voltage sense on BLACK, tapped on the TRACK side (TRACK_POS) of the switch -> PA1."
- note added: "SIGNAL DESCRIPTIONS: WHITE (+12-16V): Always-live rail from track PSU (40-90A). Powers module via F1+LDO. Also powers the TPS1212-Q1 and the anti-brake current source. BLACK (track +): Controlled by hand controller (0 to rail voltage). Falls to near 0V when controller shorts for braking. RED (common -): Braid return. Common ground reference (GND)."
- note removed: "ALL CONNECTORS: 4mm banana sockets"
- note removed: "BRAKE DETECTION (this module, not hand controller): V_BLACK < 500mV => enter brake state V_BLACK > 1500mV => exit brake state Hysteresis band prevents chatter at low throttle settings."
- note removed: "LATVIAN BRAKE (track call / emergency stop): Monitors WHITE dV/dt each 1ms tick. If WHITE drops faster than SET LATVIAN_DVDT threshold, fires immediate dead short regardless of mode or pot. Default: disabled (SET LATVIAN_DVDT 0). Recommended: SET LATVIAN_DVDT 1000 (1V/ms)."
- note removed: "SIGNAL DESCRIPTIONS: WHITE (+12-16V): Always-live rail from track PSU (40-90A capable) Powers module MCU via LDO on power supply sheet. BLACK (track +): Controlled by hand controller (0 to rail voltage). Falls to near 0V when controller shorts for braking. Module monitors dV/dt for Latvian brake feature. RED (common -): Left-hand braid return. Common ground reference."
- note removed: "Track side (J1/J3/J5) connects to the three track banana sockets. Controller side (J2/J4/J6) the hand controller plugs into. Module is inserted between track and controller. During normal running the module is fully transparent. Brake detection by voltage sense on BLACK (J3/J4) terminal."
