File: aart-brake-kicad-h/track_connectors.kicad_sch (KiCad schematic)
At the start: 0 parts

Commit message: Latest
Other:
- note added: "SIGNAL DESCRIPTIONS: WHITE (+12-16V): Always-live rail from track PSU (40-90A). Powers module via F1+LDO. Also feeds the ideal-diode gate-drive charge pump and the anti-brake current source. BLACK (track +): Controlled by hand controller (0 to rail voltage). Falls to near 0V when controller shorts for braking. RED (common -): Braid return. Common ground reference (GND)."
- note removed: "SIGNAL DESCRIPTIONS: WHITE (+12-16V): Always-live rail from track PSU (40-90A). Powers module via F1+LDO. Also powers the TPS1212-Q1 and the anti-brake current source. BLACK (track +): Controlled by hand controller (0 to rail voltage). Falls to near 0V when controller shorts for braking. RED (common -): Braid return. Common ground reference (GND)."
