File: aart-brake-kicad-h/reverse_switch.kicad_sch (KiCad schematic)
At the start: 0 parts

Commit message: Latest
Other:
- note added: "IDEAL-DIODE REVERSE BLOCK (replaces TPS1212-Q1): U5 INA210 (gain 200) senses across Rsns_sw (~1mohm). U6 LM311 compares its output to a threshold (~0.16A) with ~50mV hysteresis; on reverse current LM311 turns the gate driver off -> body diodes block. Reverse response ~2us (sim - validate with real INA210+LM311 models). The LM311 output doubles as the MCU brake-detect on PA6 (was TPS1212 I_DIR). N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"
- note added: "INSERTION DROP at 40A: 2 x 0.59mohm FET (47mV) + Rsns_sw ~1mohm (40mV) = ~87mV. Rsns_sw is a drop-vs-sense-accuracy knob: ~1mohm gives the sim +/-0.16A reverse threshold; a smaller shunt = lower drop but coarser threshold. The back-to-back pair is still required for true bidirectional blocking (a single FET body diode conducts the blocked direction)."
- note added: "PB3: now a free GPIO. The ideal diode has no enable input; the TPS1212 EN/UVLO is gone."
- note added: "Rsns_sw ~1mohm (INA210 senses)"
- note added: "TWO N-CHANNEL BIDIRECTIONAL SWITCH + IDEAL-DIODE CONTROLLER: Q5/Q6 in series, sources tied (common-source = TS). Drains to CTRL_BLACK_IN and TRACK_POS. Opposing body diodes block both directions when off; both channels conduct (low Rds) when on. Controlled as an ideal diode by U5 INA210 + U6 LM311 (+5V). GATE DRIVE OPEN ITEM: gates must be lifted above the 0-16V BLACK common source; the TPS1212 d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"
- note added: "U5 INA210 gain 200 U6 LM311 50mV hyst INA210 across Rsns_sw LM311 -> gate driver (ICs on +5V)"
- note added: "common source (TS) (gates lifted by driver)"
- note removed: "INSERTION DROP at 40A: 2 x 0.59mohm FET (47mV) + RSNS ~0.5-0.75mohm (20-30mV) = ~67-77mV. Higher than the bare-FET 47mV, but now with full protection. RSNS is a drop-vs-sense-accuracy knob; set I2t/SCP/OCP thresholds for trip above 40A (~50-60A). BONUS: a single FET cannot do reverse-block AND forward-OCP (its body diode conducts the protected direction) - the back-to-back pair is why both protec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"
- note removed: "PB3_SW_EN: optional MCU supervisory enable (EN/UVLO). Unused in Rev 11."
- note removed: "PROTECTION + REVERSE BLOCK (replaces LTC7001 + INA241 + comparator): U5 senses main-path current across RSNS (CS1+/CS1-). On reverse current it asserts I_DIR (open-drain) low; glue logic pulls INP low -> GATE off -> body diodes block. Reverse response ~6-10us (slower than a 0.75us ideal-diode controller, accepted here: the slot-car controller output stage tolerates a few us of current-limited rev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"
- note removed: "RSNS ~0.5-0.75mohm (in CS path)"
- note removed: "TWO N-CHANNEL BIDIRECTIONAL SWITCH + SMART CONTROLLER: Q5/Q6 in series, sources tied (common-source = TS/SRC). Drains to CTRL_BLACK_IN and TRACK_POS. Opposing body diodes block both directions when off; both channels conduct (low Rds) when on. U5 TPS1212-Q1 drives both gates from its GATE pin via an internal charge pump. VS ties to WHITE (3.5-73V range) so control is alive regardless of BLACK vol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"
- note removed: "U5 TPS1212-Q1 VQFN-23 VS=WHITE GATE->Q5/Q6 gates CS1+/CS1- across RSNS"
- note removed: "common source (TS) -> TPS1212 SRC"
- title: AART Brake Module — 7: Reverse-Blocking Pass Switch (two N-channel + TPS1212-Q1) -> AART Brake Module — 7: Reverse-Blocking Pass Switch (two N-channel + INA210/LM311 ideal diode)
